File: elixir-sensors.kicad_sch (KiCad schematic)
At the start: 75 parts, among them J16 Conn_02x05_Odd_Even, J17 02x04, J5 Conn_01x03_Pin, Q1 BC847, SW4 SW_Push, SW6 SW_Push, U10 PCF85063ATL, U11 SN74AUC1G66DBVR, U15 ESP32-C3-MINI-1-N4, U16 AP2171W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

Commit message: Move ATECC to rev C. Fixes #2.
Parts:
- U7: value ATECC608A-MAHDA -> ATECC608C; Link1 https://www.digikey.com/en/products/detail/microchip-technology/ATECC608A-MAHDA-S/7928113 -> https://www.digikey.com/en/products/detail/microchip-technology/ATECC608C-MAHDA-T/21668937; MPN1 ATECC608A-MAHDA-S -> ATECC608C-MAHDA-T
Changed lines of the file:
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@@
 	(label "C3_IO10"
 		(at 69.215 132.08 0)
-		(fields_autoplaced yes)
 		(effects
 			(font
@@
 	(label "C3_IO2"
 		(at 69.215 137.16 0)
-		(fields_autoplaced yes)
 		(effects
 			(font
@@
 	(label "C3_USB_P"
 		(at 129.54 58.42 180)
-		(fields_autoplaced yes)
 		(effects
 			(font
@@
 	(label "C3_IO3"
 		(at 99.06 137.16 180)
-		(fields_autoplaced yes)
 		(effects
 			(font
@@
 	(label "C3_IO7"
 		(at 69.215 127 0)
-		(fields_autoplaced yes)
 		(effects
 			(font
@@
 	(label "C3_IO6"
 		(at 99.06 129.54 180)
-		(fields_autoplaced yes)
 		(effects
 			(font
@@
 	(label "C3_IO0"
 		(at 69.215 134.62 0)
-		(fields_autoplaced yes)
 		(effects
 			(font
@@
 	(label "C3_USB_N"
 		(at 59.055 113.03 0)
-		(fields_autoplaced yes)
 		(effects
 			(font
@@
 	(label "ESP32-C3-RX-PROG"
 		(at 62.23 68.58 0)
-		(fields_autoplaced yes)
 		(effects
 			(font
@@
 	(label "C3_IO5"
 		(at 76.835 60.96 0)
-		(fields_autoplaced yes)
 		(effects
 			(font
@@
 	(label "C3_IO2"
 		(at 76.835 53.34 0)
-		(fields_autoplaced yes)
 		(effects
 			(font
@@
 	(label "SWITCHED_PWR_I2C"
 		(at 333.375 118.11 0)
-		(fields_autoplaced yes)
 		(effects
 			(font
@@
 	(label "C3_IO8"
 		(at 98.425 127 180)
-		(fields_autoplaced yes)
 		(effects
 			(font
@@
 	(label "ESP32-C3-RX-PROG"
 		(at 59.055 107.95 0)
-		(fields_autoplaced yes)
 		(effects
 			(font
@@
 	(label "C3_IO7"
 		(at 129.54 48.26 180)
-		(fields_autoplaced yes)
 		(effects
 			(font
@@
 	(label "C3_USB_P"
 		(at 118.11 113.03 180)
-		(fields_autoplaced yes)
 		(effects
 			(font
@@
 	(label "C3_IO10"
 		(at 129.54 55.88 180)
-		(fields_autoplaced yes)
 		(effects
 			(font
@@
 	(label "ESP32-C3-TX-PROG"
 		(at 59.055 110.49 0)
-		(fields_autoplaced yes)
 		(effects
 			(font
@@
 	(label "C3_IO1"
 		(at 99.06 134.62 180)
-		(fields_autoplaced yes)
 		(effects
 			(font
@@
 	(label "BME280_3V3"
 		(at 71.12 200.66 0)
-		(fields_autoplaced yes)
 		(effects
 			(font
@@
 	(label "SWITCHED_PWR_I2C"
 		(at 279.4 57.15 0)
-		(fields_autoplaced yes)
 		(effects
 			(font
@@
 	(label "C3_IO0"
 		(at 76.835 48.26 0)
-		(fields_autoplaced yes)
 		(effects
 			(font
@@
 	(label "C3_IO4"
 		(at 99.06 132.08 180)
-		(fields_autoplaced yes)
 		(effects
 			(font
@@
 	(label "C3_IO3"
 		(at 76.835 55.88 0)
-		(fields_autoplaced yes)
 		(effects
 			(font
@@
 	(label "C3_IO9"
 		(at 118.11 110.49 180)
-		(fields_autoplaced yes)
 		(effects
 			(font
@@
 	(label "C3_USB_N"
 		(at 129.54 60.96 180)
-		(fields_autoplaced yes)
 		(effects
 			(font
@@
 	(label "C3_IO6"
 		(at 76.835 63.5 0)
-		(fields_autoplaced yes)
 		(effects
 			(font
@@
 	(label "C3_IO5"
 		(at 69.215 129.54 0)
-		(fields_autoplaced yes)
 		(effects
 			(font
@@
 	(label "ESP32-C3-TX-PROG"
 		(at 62.23 71.12 0)
-		(fields_autoplaced yes)
 		(effects
 			(font
@@
 	(label "C3_IO1"
 		(at 76.835 50.8 0)
-		(fields_autoplaced yes)
 		(effects
 			(font
@@
 	(label "BME280_3V3"
 		(at 80.645 231.14 180)
-		(fields_autoplaced yes)
 		(effects
 			(font
@@
 	(label "C3_IO9"
 		(at 167.005 52.705 0)
-		(fields_autoplaced yes)
 		(effects
 			(font
@@
 	(label "SWITCHED_PWR_I2C"
 		(at 240.665 118.11 0)
-		(fields_autoplaced yes)
 		(effects
 			(font
@@
 	(label "C3_IO4"
 		(at 76.835 58.42 0)
-		(fields_autoplaced yes)
 		(effects
 			(font
@@
 	(label "C3_IO8"
 		(at 129.54 50.8 180)
-		(fields_autoplaced yes)
 		(effects
 			(font
@@
 			)
 		)
-		(property "Value" "ATECC608A-MAHDA"
+		(property "Value" "ATECC608C"
 			(at 191.77 160.02 0)
 			(effects
@@
 			)
 		)
-		(property "Link1" "https://www.digikey.com/en/products/detail/microchip-technology/ATECC608A-MAHDA-S/7928113"
+		(property "Link1" "https://www.digikey.com/en/products/detail/microchip-technology/ATECC608C-MAHDA-T/21668937"
 			(at 198.12 158.75 0)
 			(effects
@@
 			)
 		)
-		(property "MPN1" "ATECC608A-MAHDA-S"
+		(property "MPN1" "ATECC608C-MAHDA-T"
 			(at 198.12 158.75 0)
 			(effects
